File: wirewarp board v3/wirewarp board v3.kicad_pcb (KiCad board)
At the start: 2 copper layers, 99.1 x 99.1 mm, 1375 parts

Commit message: review of kicad files
Other:
- board text added: "pwr"
- board text removed: "J"
- board text removed: "K"
- board text removed: "sk"

Commit message: update version 3 of 10x10 protoboard
Parts:
- removed the ? at (69.8, 146.1) (x2)
- removed the ? at (105.4, 146.1) (x2)
- removed the ? at (120.7, 146.1) (x2)
- removed the ? at (95.2, 146.1) (x2)
- removed the ? at (130.8, 146.1) (x2)
- removed the ? at (80.0, 146.1) (x2)
- added ?: , , F.Cu at (34.3, 134.5)
- added ?: , , F.Cu at (34.3, 106.6)
- added ?: , , F.Cu at (34.3, 116.7)
- added ?: , , F.Cu at (34.3, 114.2)
- added ?: , , F.Cu at (34.3, 48.1)
- added ?: , , F.Cu at (34.3, 91.3)
- added ?: , , F.Cu at (34.3, 81.2)
- added ?: , , F.Cu at (34.3, 71.0)
- added ?: , , F.Cu at (95.2, 146.1)
- added ?: , , F.Cu at (80.0, 146.1)
- added ?: , , F.Cu at (34.3, 129.4)
- added ?: , , F.Cu at (34.3, 119.3)
- added ?: , , F.Cu at (34.3, 68.5)
- added ?: , , F.Cu at (105.4, 146.1)
- added ?: , , F.Cu at (34.3, 58.3)
- added ?: , , F.Cu at (69.8, 146.1)
- added ?: , , F.Cu at (34.3, 83.7)
- added ?: , , F.Cu at (34.3, 88.8)
- added ?: , , F.Cu at (34.3, 53.2)
- added ?: , , F.Cu at (34.3, 139.6)
- added ?: , , F.Cu at (130.8, 146.1)
- added ?: , , F.Cu at (34.3, 93.9)
- added ?: , , F.Cu at (34.3, 65.9)
- added ?: , , F.Cu at (34.3, 86.2)
- added ?: , , F.Cu at (34.3, 104.0)
- added ?: , , F.Cu at (34.3, 63.4)
- added ?: , , F.Cu at (34.3, 73.5)
- added ?: , , F.Cu at (34.3, 126.9)
- added ?: , , F.Cu at (34.3, 109.1)
- added ?: , , F.Cu at (34.3, 124.3)
- added ?: , , F.Cu at (34.3, 121.8)
- added ?: , , F.Cu at (34.3, 111.6)
- added ?: , , F.Cu at (34.3, 76.1)
- added ?: , , F.Cu at (34.3, 96.4)
- added ?: , , F.Cu at (34.3, 101.5)
- added ?: , , F.Cu at (34.3, 60.8)
- added ?: , , F.Cu at (34.3, 137.0)
- added ?: , , F.Cu at (34.3, 55.8)
- added ?: , , F.Cu at (34.3, 78.6)
- added ?: , , F.Cu at (34.3, 50.7)
- added ?: , , F.Cu at (34.3, 132.0)
- added ?: , , F.Cu at (120.7, 146.1)
- added ?: , , F.Cu at (34.3, 98.9)
Routing:
- net (no net): track 2872.7 -> 2884.2 mm
Other:
- outline, holes or cut-outs redrawn
- board text added: "conL"
- board text added: "conR"
- board text removed: "CONL"
- board text removed: "CONR"
- board text removed: "ww"

Commit message: update of 10x10 protoboards, conn connected
Routing:
- net (no net): track 2884.2 -> 6659.2 mm
